File: _autosave-Senior_Design.kicad_pcb (KiCad board)
At the start: 2 copper layers, 100 x 100 mm, 158 parts, among them J1001 GS2, J102 GS2, J103 BARREL_JACK, J104 ISP, J1201 USB_A, J1202 USB_A, J1401 USB_OTG, J1402 GS2, J1403 GS2, J1404 GS3, Q1001 MMBT4403, Q101 Q_NMOS_DGS, Q1101 Q_NMOS_DGS, Q1102 Q_PMOS_DGS, Q601 Q_NMOS_DGS, Q602 Q_PMOS_DGS, U1001 HX711, U101 ATMEGA2561-16AU, U1101 MOUDLE-BLUETOOTH-HC-05(34P-27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, U1301 LM358_IC, U1401 FT231XS, U1501 TPS562210, U1701 INA169, U1801 INA169, U1901 INA169, U201 TPS562210, U301 TPS562210, Y101 16MHZ

Commit message: hc-05 and buzzer 3d model
Parts:
- moved J1401 1.50 mm to (135.0, 53.0)
Changed lines of the file:
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@@
   (general
     (links 308)
-    (no_connects 246)
+    (no_connects 247)
     (area 49.924999 49.924999 150.075001 150.075001)
     (thickness 1.6)
@@
     (pad 1 thru_hole circle (at -5.08 0) (size 2.49936 2.49936) (drill 1.00076) (layers *.Cu *.Mask)
       (net 2 5V-BUS))
+    (model ../../../../../../Users/Chase/Documents/KiCAD/Senior_Design/lib/PB-0627PE.wrl
+      (at (xyz 0 0 0))
+      (scale (xyz 1000 1000 1000))
+      (rotate (xyz 0 0 0))
+    )
   )
   (module Capacitors_SMD:C_0603 (layer F.Cu)
@@
   )
   (module Connectors:USB_Micro-B (layer F.Cu)
-    (at 135 54.5 180)
+    (at 135 53 180)
     (descr "Micro USB Type B Receptacle")
     (tags "USB USB_B USB_micro USB_OTG")
@@
     (pad 6 thru_hole oval (at 3.5 1.35 270) (size 1.55 1) (drill oval 1.15 0.5) (layers *.Cu *.Mask)
       (net 56 "Net-(J1401-Pad6)"))
+    (model C:/Users/Chase/Documents/KiCAD/Senior_Design/lib/Molex_Mirco_USB_105017-0001.wrl
+      (at (xyz 0 0.1 0))
+      (scale (xyz 1 1 1))
+      (rotate (xyz 0 0 0))
+    )
   )
   (module Connectors:GS2 (layer F.Cu)
@@
     (pad 34 smd rect (at 6.5 -6.5 90) (size 2 1) (layers F.Cu F.Paste F.Mask)
       (net 76 "Net-(R1105-Pad2)"))
+    (model C:/Users/Chase/Documents/KiCAD/Senior_Design/lib/bluetooth.wrl
+      (at (xyz 0 0 0))
+      (scale (xyz 400 400 400))
+      (rotate (xyz 270 0 270))
+    )
   )
   (module Connectors:Pin_d1.3mm_L11.0mm (layer F.Cu)
